Commit message: 优化仿真页面；修正坐标顺序（xyzw）

File: assets/Tienkung/urdf/walker_tienkung_ei.urdf (robot description, URDF)
Before this commit: robot humanoid, 34 links, 33 joints
Links:
- link ankle_pitch_l_link: geometry collision mesh filename=package://walker_tienkung_ei_description/meshes/ankle_pitch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; visual mesh filename=package://walker_tienkung_ei_description/meshes/ankle_pitch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
- link ankle_pitch_r_link: geometry collision mesh filename=package://walker_tienkung_ei_description/meshes/ankle_pitch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; visual mesh filename=package://walker_tienkung_ei_description/meshes/ankle_pitch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
- link ankle_roll_l_link: geometry collision mesh filename=package://walker_tienkung_ei_description/meshes/ankle_roll_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; visual mesh filename=package://walker_tienkung_ei_description/meshes/ankle_roll_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
- link ankle_roll_r_link: geometry collision mesh filename=package://walker_tienkung_ei_description/meshes/ankle_roll_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; visual mesh filename=package://walker_tienkung_ei_description/meshes/ankle_roll_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
- link camera_body_back_link: geometry collision mesh filename=package://walker_tienkung_ei_description/meshes/camera_body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; visual mesh filename=package://walker_tienkung_ei_description/meshes/camera_body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
- link camera_body_front_link: geometry collision mesh filename=package://walker_tienkung_ei_description/meshes/camera_body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; visual mesh filename=package://walker_tienkung_ei_description/meshes/camera_body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
- link camera_head_link: geometry collision mesh filename=package://walker_tienkung_ei_description/meshes/camera_head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; visual mesh filename=package://walker_tienkung_ei_description/meshes/camera_head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
- link elbow_pitch_l_link: geometry collision mesh filename=package://walker_tienkung_ei_description/meshes/elbow_pitch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; visual mesh filename=package://walker_tienkung_ei_description/meshes/elbow_pitch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
- link elbow_pitch_r_link: geometry collision mesh filename=package://walker_tienkung_ei_description/meshes/elbow_pitch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; visual mesh filename=package://walker_tienkung_ei_description/meshes/elbow_pitch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
- link elbow_yaw_l_link: geometry collision mesh filename=package://walker_tienkung_ei_description/meshes/elbow_yaw_l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; visual mesh filename=package://walker_tienkung_ei_description/meshes/elbow_yaw_l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
- link elbow_yaw_r_link: geometry collision mesh filename=package://walker_tienkung_ei_description/meshes/elbow_yaw_r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; visual mesh filename=package://walker_tienkung_ei_description/meshes/elbow_yaw_r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
- link head_pitch_link: geometry collision mesh filename=package://walker_tienkung_ei_description/meshes/head_pitch_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; visual mesh filename=package://walker_tienkung_ei_description/meshes/head_pitch_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
- link head_roll_link: geometry collision mesh filename=package://walker_tienkung_ei_description/meshes/head_roll_l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; visual mesh filename=package://walker_tienkung_ei_description/meshes/head_roll_l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
- link head_yaw_link: geometry collision mesh filename=package://walker_tienkung_ei_description/meshes/head_yaw_li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; visual mesh filename=package://walker_tienkung_ei_description/meshes/head_yaw_li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
- link hip_pitch_l_link: geometry collision mesh filename=package://walker_tienkung_ei_description/meshes/hip_pitch_l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; visual mesh filename=package://walker_tienkung_ei_description/meshes/hip_pitch_l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
- link hip_pitch_r_link: geometry collision mesh filename=package://walker_tienkung_ei_description/meshes/hip_pitch_r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; visual mesh filename=package://walker_tienkung_ei_description/meshes/hip_pitch_r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
- link hip_roll_l_link: geometry collision mesh filename=package://walker_tienkung_ei_description/meshes/hip_roll_l_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; visual mesh filename=package://walker_tienkung_ei_description/meshes/hip_roll_l_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
- link hip_roll_r_link: geometry collision mesh filename=package://walker_tienkung_ei_description/meshes/hip_roll_r_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; visual mesh filename=package://walker_tienkung_ei_description/meshes/hip_roll_r_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
- link hip_yaw_l_link: geometry collision mesh filename=package://walker_tienkung_ei_description/meshes/hip_yaw_l_l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; visual mesh filename=package://walker_tienkung_ei_description/meshes/hip_yaw_l_l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
- link hip_yaw_r_link: geometry collision mesh filename=package://walker_tienkung_ei_description/meshes/hip_yaw_r_l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; visual mesh filename=package://walker_tienkung_ei_description/meshes/hip_yaw_r_l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
- link knee_pitch_l_link: geometry collision mesh filename=package://walker_tienkung_ei_description/meshes/knee_pitch_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; visual mesh filename=package://walker_tienkung_ei_description/meshes/knee_pitch_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
- link knee_pitch_r_link: geometry collision mesh filename=package://walker_tienkung_ei_description/meshes/knee_pitch_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; visual mesh filename=package://walker_tienkung_ei_description/meshes/knee_pitch_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
- link pelvis: geometry collision mesh filename=package://walker_tienkung_ei_description/meshes/pelvis.STL; visual mesh filename=package://walker_tienkung_ei_description/meshes/pelvis.STL
- link shoulder_pitch_l_link: geometry collision mesh filename=package://walker_tienkung_ei_description/meshes/shoulder_pi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; visual mesh filename=package://walker_tienkung_ei_description/meshes/shoulder_pi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
- link shoulder_pitch_r_link: geometry collision mesh filename=package://walker_tienkung_ei_description/meshes/shoulder_pi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; visual mesh filename=package://walker_tienkung_ei_description/meshes/shoulder_pi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
- link shoulder_roll_l_link: geometry collision mesh filename=package://walker_tienkung_ei_description/meshes/shoulder_ro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; visual mesh filename=package://walker_tienkung_ei_description/meshes/shoulder_ro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
- link shoulder_roll_r_link: geometry collision mesh filename=package://walker_tienkung_ei_description/meshes/shoulder_ro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; visual mesh filename=package://walker_tienkung_ei_description/meshes/shoulder_ro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
- link shoulder_yaw_l_link: geometry collision mesh filename=package://walker_tienkung_ei_description/meshes/shoulder_ya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; visual mesh filename=package://walker_tienkung_ei_description/meshes/shoulder_ya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
- link shoulder_yaw_r_link: geometry collision mesh filename=package://walker_tienkung_ei_description/meshes/shoulder_ya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; visual mesh filename=package://walker_tienkung_ei_description/meshes/shoulder_ya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
- link waist_yaw_link: geometry collision mesh filename=package://walker_tienkung_ei_description/meshes/waist_yaw_l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; visual mesh filename=package://walker_tienkung_ei_description/meshes/waist_yaw_l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
- link wrist_pitch_l_link: geometry collision mesh filename=package://walker_tienkung_ei_description/meshes/wrist_pitch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; visual mesh filename=package://walker_tienkung_ei_description/meshes/wrist_pitch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
- link wrist_pitch_r_link: geometry collision mesh filename=package://walker_tienkung_ei_description/meshes/wrist_pitch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; visual mesh filename=package://walker_tienkung_ei_description/meshes/wrist_pitch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
- link wrist_roll_l_link: geometry collision mesh filename=package://walker_tienkung_ei_description/meshes/wrist_roll_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; visual mesh filename=package://walker_tienkung_ei_description/meshes/wrist_roll_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
- link wrist_roll_r_link: geometry collision mesh filename=package://walker_tienkung_ei_description/meshes/wrist_roll_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; visual mesh filename=package://walker_tienkung_ei_description/meshes/wrist_roll_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

Commit message: 适配新urdf，虽然仿真仍无法正常显示，但不影响训练
- 将 URDF 中的 mesh 路径从 package:// 改为仓库内相对路径，保证非 ROS 环境下可正常加载
- 将多个 link 的 collision 从原始 mesh 改为 box，并补充对应 origin/size，降低复杂碰撞带来的仿真不稳定
- 调整腿部部分关节的父子关系与 joint origin，用于对齐天工机器人的实际运动链定义
- 注释掉相机相关固定 link/joint，减少无关刚体对仿真和索引映射的干扰
- 更新 FK XML 的 meshdir 配置，并将部分 mesh 切换为 *_mujoco.STL，以匹配 MuJoCo/FK 使用的几何文件
- 移除 XML 中不必要的 apirate 选项，提升配置兼容性

File: assets/Tienkung/urdf/walker_tienkung_ei.urdf (robot description, URDF)
Before this commit: robot humanoid, 34 links, 33 joints
Links:
- removed link camera_body_back_link
- removed link camera_body_front_link
- removed link camera_head_link
- link ankle_pitch_l_link: geometry collision box size=0.059400 0.059400 0.021600; visual mesh filename=../meshes/ankle_pitch_l_link.STL
- link ankle_pitch_r_link: geometry collision box size=0.059400 0.059400 0.021600; visual mesh filename=../meshes/ankle_pitch_r_link.STL
- link ankle_roll_l_link: geometry collision box size=0.253435 0.105883 0.085941; visual mesh filename=../meshes/ankle_roll_l_link.STL
- link ankle_roll_r_link: geometry collision box size=0.253435 0.105883 0.085941; visual mesh filename=../meshes/ankle_roll_r_link.STL
- link elbow_pitch_l_link: geometry collision box size=0.084123 0.098719 0.091021; visual mesh filename=../meshes/elbow_pitch_l_link.STL
- link elbow_pitch_r_link: geometry collision box size=0.084123 0.098719 0.091021; visual mesh filename=../meshes/elbow_pitch_r_link.STL
- link elbow_yaw_l_link: geometry collision box size=0.070769 0.099862 0.199759; visual mesh filename=../meshes/elbow_yaw_l_link.STL
- link elbow_yaw_r_link: geometry collision box size=0.070769 0.099862 0.199759; visual mesh filename=../meshes/elbow_yaw_r_link.STL
- link head_pitch_link: geometry collision box size=0.069514 0.068940 0.059773; visual mesh filename=../meshes/head_pitch_link.STL
- link head_roll_link: geometry collision box size=0.242521 0.151702 0.235080; visual mesh filename=../meshes/head_roll_link.STL
- link head_yaw_link: geometry collision box size=0.100397 0.090342 0.083758; visual mesh filename=../meshes/head_yaw_link.STL
- link hip_pitch_l_link: geometry collision box size=0.155999 0.107960 0.164880; visual mesh filename=../meshes/hip_pitch_l_link.STL
- link hip_pitch_r_link: geometry collision box size=0.156028 0.107964 0.164880; visual mesh filename=../meshes/hip_pitch_r_link.STL
- link hip_roll_l_link: geometry collision box size=0.176494 0.110621 0.112739; visual mesh filename=../meshes/hip_roll_l_link.STL
- link hip_roll_r_link: geometry collision box size=0.176494 0.110621 0.112739; visual mesh filename=../meshes/hip_roll_r_link.STL
- link hip_yaw_l_link: geometry collision box size=0.155887 0.141082 0.309206; visual mesh filename=../meshes/hip_yaw_l_link.STL
- link hip_yaw_r_link: geometry collision box size=0.155855 0.141082 0.309265; visual mesh filename=../meshes/hip_yaw_r_link.STL
- link knee_pitch_l_link: geometry collision box size=0.084733 0.083538 0.424877; visual mesh filename=../meshes/knee_pitch_l_link.STL
- link knee_pitch_r_link: geometry collision box size=0.084733 0.083552 0.424877; visual mesh filename=../meshes/knee_pitch_r_link.STL
- link pelvis: geometry collision box size=0.219663 0.172732 0.159129; visual mesh filename=../meshes/pelvis.STL
- link shoulder_pitch_l_link: geometry collision box size=0.089370 0.108115 0.081526; visual mesh filename=../meshes/shoulder_pitch_l_link.STL
- link shoulder_pitch_r_link: geometry collision box size=0.089370 0.108115 0.081526; visual mesh filename=../meshes/shoulder_pitch_r_link.STL
- link shoulder_roll_l_link: geometry collision box size=0.102233 0.103086 0.145652; visual mesh filename=../meshes/shoulder_roll_l_link.STL
- link shoulder_roll_r_link: geometry collision box size=0.102233 0.103086 0.145652; visual mesh filename=../meshes/shoulder_roll_r_link.STL
- link shoulder_yaw_l_link: geometry collision box size=0.089051 0.104139 0.222196; visual mesh filename=../meshes/shoulder_yaw_l_link.STL
- link shoulder_yaw_r_link: geometry collision box size=0.089051 0.104139 0.222196; visual mesh filename=../meshes/shoulder_yaw_r_link.STL
- link waist_yaw_link: geometry collision box size=0.254932 0.292847 0.514330; visual mesh filename=../meshes/waist_yaw_link.STL
- link wrist_pitch_l_link: geometry collision box size=0.070290 0.061385 0.053836; visual mesh filename=../meshes/wrist_pitch_l_link.STL
- link wrist_pitch_r_link: geometry collision box size=0.070290 0.061385 0.053836; visual mesh filename=../meshes/wrist_pitch_r_link.STL
- link wrist_roll_l_link: geometry collision box size=0.073159 0.061803 0.066398; visual mesh filename=../meshes/wrist_roll_l_link.STL
- link wrist_roll_r_link: geometry collision box size=0.073159 0.061803 0.066398; visual mesh filename=../meshes/wrist_roll_r_link.STL
Joints:
- removed joint camera_body_back_joint
- removed joint camera_body_front_joint
- removed joint camera_head_joint
- joint hip_pitch_l_joint: origin xyz=0 0.122 -0.046 rpy=0 0 0 -> xyz=0 0.094 0.0987 rpy=0 0 0; parent hip_roll_l_link -> hip_yaw_l_link
- joint hip_pitch_r_joint: origin xyz=0 -0.122 -0.046 rpy=0 0 0 -> xyz=0 -0.094 0.0987 rpy=0 0 0; parent hip_roll_r_link -> hip_yaw_r_link
- joint hip_yaw_l_joint: origin xyz=0 0 -0.0987 rpy=0 0 0 -> xyz=0 0.028 -0.1317 rpy=0 0 0; parent hip_pitch_l_link -> hip_roll_l_link
- joint hip_yaw_r_joint: origin xyz=0 0 -0.0987 rpy=0 0 0 -> xyz=0 -0.028 -0.1317 rpy=0 0 0; parent hip_pitch_r_link -> hip_roll_r_link
- joint knee_pitch_l_joint: origin xyz=0 -4.2833E-05 -0.3013 rpy=0 0 0 -> xyz=0 0 -0.413 rpy=0 0 0; parent hip_yaw_l_link -> hip_pitch_l_link
- joint knee_pitch_r_joint: origin xyz=0 0.00015001 -0.3013 rpy=0 0 0 -> xyz=0 0 -0.413 rpy=0 0 0; parent hip_yaw_r_link -> hip_pitch_r_link
